File: PCB Designs/ES_001 PCB BMS/BMS12v3.kicad_pcb (KiCad board)
At the start: 2 copper layers, 61 x 61 mm, 85 parts, among them IC2 78LXXSOT89, Q1 CRYSTALCTS406

Commit message: Generated gerber files for BMS Zeva
Parts:
- added G***: LOGO, Logo_ISC:LogoISC, B.Cu at (147.3, 111.8)
Other:
- board text added: "ZEVA BMS 01/23 F. de Paz R. Morán"
